File: keyboard1.kicad_pcb (KiCad board)
At the start: 2 copper layers, 88.9 x 41.9 mm, 4 parts, among them SW1 SW_Push

Commit message: pcb progress
Parts:
- removed BT1: Battery, Battery:BatteryHolder_Keystone_2462_2xAA
- added '1: SW_Push, Button_Switch_Keyboard:SW_Cherry_MX1A_1.00u_PCB, F.Cu at (309.2, 128.3)
- added ,1: SW_Push, Button_Switch_Keyboard:SW_Cherry_MX1A_1.00u_PCB, F.Cu at (257.8, 148.6)
- added -1: SW_Push, Button_Switch_Keyboard:SW_Cherry_MX1A_1.00u_PCB, F.Cu at (294.6, 87.6)
- added .1: SW_Push, Button_Switch_Keyboard:SW_Cherry_MX1A_1.00u_PCB, F.Cu at (278.1, 148.6)
- added /1: SW_Push, Button_Switch_Keyboard:SW_Cherry_MX1A_1.00u_PCB, F.Cu at (298.4, 148.6)
- added ;1: SW_Push, Button_Switch_Keyboard:SW_Cherry_MX1A_1.00u_PCB, F.Cu at (288.9, 128.3)
- added =1: SW_Push, Button_Switch_Keyboard:SW_Cherry_MX1A_1.00u_PCB, F.Cu at (315.0, 87.6)
- added ALT_LEFT1: SW_Push, Button_Switch_Keyboard:SW_Cherry_MX1A_1.25u_PCB, F.Cu at (124.5, 168.9)
- added ALT_RIGHT1: SW_Push, Button_Switch_Keyboard:SW_Cherry_MX1A_1.25u_PCB, F.Cu at (269.2, 168.9)
- added ARROW_DOWN1: SW_Push, Button_Switch_Keyboard:SW_Cherry_MX1A_1.00u_PCB, F.Cu at (312.4, 168.9)
- added ARROW_LEFT1: SW_Push, Button_Switch_Keyboard:SW_Cherry_MX1A_1.00u_PCB, F.Cu at (292.1, 168.9)
- added ARROW_RIGHT1: SW_Push, Button_Switch_Keyboard:SW_Cherry_MX1A_1.00u_PCB, F.Cu at (332.7, 168.9)
- added ARROW_UP1: SW_Push, Button_Switch_Keyboard:SW_Cherry_MX1A_1.00u_PCB, F.Cu at (318.8, 148.6)
- added BACKSPACE1: SW_Push, Button_Switch_Keyboard:SW_Cherry_MX1A_2.00u_PCB, F.Cu at (344.9, 87.6)
- added C1: 22p, Capacitor_SMD:C_1812_4532Metric_Pad1.30x3.40mm_HandSolder, B.Cu at (156.2, 179.1)
- added C2: 1u, Capacitor_SMD:C_1812_4532Metric_Pad1.30x3.40mm_HandSolder, B.Cu at (212.1, 177.8)
- added C3: 22p, Capacitor_SMD:C_1812_4532Metric_Pad1.30x3.40mm_HandSolder, B.Cu at (172.7, 179.1)
- added CTRL1: SW_Push, Button_Switch_Keyboard:SW_Cherry_MX1A_1.25u_PCB, F.Cu at (73.7, 168.9)
- added D10: DIODE, Diode_SMD:D_1206_3216Metric, B.Cu at (97.8, 179.1)
- added D11: DIODE, Diode_SMD:D_1206_3216Metric, B.Cu at (109.2, 97.8)
- added D12: DIODE, Diode_SMD:D_1206_3216Metric, B.Cu at (120.7, 118.1)
- added D13: DIODE, Diode_SMD:D_1206_3216Metric, B.Cu at (125.1, 138.4)
- added D14: DIODE, Diode_SMD:D_1206_3216Metric, B.Cu at (114.3, 158.8)
- added D15: DIODE, Diode_SMD:D_1206_3216Metric, B.Cu at (123.2, 179.1)
- added D16: DIODE, Diode_SMD:D_1206_3216Metric, B.Cu at (129.5, 97.8)
- added D17: DIODE, Diode_SMD:D_1206_3216Metric, B.Cu at (141.0, 118.1)
- added D18: DIODE, Diode_SMD:D_1206_3216Metric, B.Cu at (145.4, 138.4)
- added D19: DIODE, Diode_SMD:D_1206_3216Metric, B.Cu at (134.6, 158.8)
- added D2: DIODE, Diode_SMD:D_1206_3216Metric, B.Cu at (68.6, 97.8)
- added D20: DIODE, Diode_SMD:D_1206_3216Metric, B.Cu at (149.9, 97.8)
- added D21: DIODE, Diode_SMD:D_1206_3216Metric, B.Cu at (161.3, 118.1)
- added D22: DIODE, Diode_SMD:D_1206_3216Metric, B.Cu at (165.7, 138.4)
- added D23: DIODE, Diode_SMD:D_1206_3216Metric, B.Cu at (154.9, 158.8)
- added D24: DIODE, Diode_SMD:D_1206_3216Metric, B.Cu at (170.2, 97.8)
- added D25: DIODE, Diode_SMD:D_1206_3216Metric, B.Cu at (181.6, 118.1)
- added D26: DIODE, Diode_SMD:D_1206_3216Metric, B.Cu at (186.1, 138.4)
- added D27: DIODE, Diode_SMD:D_1206_3216Metric, B.Cu at (175.3, 158.8)
- added D28: DIODE, Diode_SMD:D_1206_3216Metric, B.Cu at (190.5, 97.8)
- added D29: DIODE, Diode_SMD:D_1206_3216Metric, B.Cu at (201.9, 118.1)
- added D3: DIODE, Diode_SMD:D_1206_3216Metric, B.Cu at (74.9, 118.1)
- added D30: DIODE, Diode_SMD:D_1206_3216Metric, B.Cu at (206.4, 138.4)
- added D31: DIODE, Diode_SMD:D_1206_3216Metric, B.Cu at (195.6, 158.8)
- added D32: DIODE, Diode_SMD:D_1206_3216Metric, B.Cu at (195.6, 177.8)
- added D33: DIODE, Diode_SMD:D_1206_3216Metric, B.Cu at (210.8, 97.8)
- added D34: DIODE, Diode_SMD:D_1206_3216Metric, B.Cu at (222.2, 118.1)
- added D35: DIODE, Diode_SMD:D_1206_3216Metric, B.Cu at (226.7, 138.4)
- added D36: DIODE, Diode_SMD:D_1206_3216Metric, B.Cu at (215.9, 158.8)
- added D37: DIODE, Diode_SMD:D_1206_3216Metric, B.Cu at (231.1, 97.8)
- added D38: DIODE, Diode_SMD:D_1206_3216Metric, B.Cu at (242.6, 118.1)
- added D39: DIODE, Diode_SMD:D_1206_3216Metric, B.Cu at (247.0, 138.4)
- added D4: DIODE, Diode_SMD:D_1206_3216Metric, B.Cu at (76.2, 138.4)
- added D40: DIODE, Diode_SMD:D_1206_3216Metric, B.Cu at (236.2, 158.8)
- added D41: DIODE, Diode_SMD:D_1206_3216Metric, B.Cu at (251.5, 97.8)
- added D42: DIODE, Diode_SMD:D_1206_3216Metric, B.Cu at (262.9, 118.1)
- added D43: DIODE, Diode_SMD:D_1206_3216Metric, B.Cu at (267.3, 138.4)
- added D44: DIODE, Diode_SMD:D_1206_3216Metric, B.Cu at (256.5, 158.8)
- added D45: DIODE, Diode_SMD:D_1206_3216Metric, B.Cu at (271.8, 97.8)
- added D46: DIODE, Diode_SMD:D_1206_3216Metric, B.Cu at (283.2, 118.1)
- added D47: DIODE, Diode_SMD:D_1206_3216Metric, B.Cu at (287.7, 138.4)
- added D48: DIODE, Diode_SMD:D_1206_3216Metric, B.Cu at (276.9, 158.8)
- added D49: DIODE, Diode_SMD:D_1206_3216Metric, B.Cu at (268.0, 179.1)
- added D5: DIODE, Diode_SMD:D_1206_3216Metric, B.Cu at (81.3, 158.8)
- added D50: DIODE, Diode_SMD:D_1206_3216Metric, B.Cu at (292.1, 97.8)
- added D51: DIODE, Diode_SMD:D_1206_3216Metric, B.Cu at (303.5, 118.1)
- added D52: DIODE, Diode_SMD:D_1206_3216Metric, B.Cu at (308.0, 138.4)
- added D53: DIODE, Diode_SMD:D_1206_3216Metric, B.Cu at (297.2, 158.8)
- added D54: DIODE, Diode_SMD:D_1206_3216Metric, B.Cu at (290.8, 179.1)
- added D55: DIODE, Diode_SMD:D_1206_3216Metric, B.Cu at (312.4, 97.8)
- added D56: DIODE, Diode_SMD:D_1206_3216Metric, B.Cu at (323.9, 118.1)
- added D57: DIODE, Diode_SMD:D_1206_3216Metric, B.Cu at (340.4, 138.4)
- added D58: DIODE, Diode_SMD:D_1206_3216Metric, B.Cu at (317.5, 158.8)
- added D59: DIODE, Diode_SMD:D_1206_3216Metric, B.Cu at (311.1, 179.1)
- added D6: DIODE, Diode_SMD:D_1206_3216Metric, B.Cu at (72.4, 179.1)
- added D60: DIODE, Diode_SMD:D_1206_3216Metric, B.Cu at (342.9, 97.8)
- added D61: DIODE, Diode_SMD:D_1206_3216Metric, B.Cu at (349.2, 118.1)
- added D62: DIODE, Diode_SMD:D_1206_3216Metric, B.Cu at (345.4, 158.8)
- added D63: DIODE, Diode_SMD:D_1206_3216Metric, B.Cu at (331.5, 179.1)
- added D7: DIODE, Diode_SMD:D_1206_3216Metric, B.Cu at (88.9, 97.8)
- added D8: DIODE, Diode_SMD:D_1206_3216Metric, B.Cu at (100.3, 118.1)
- added D9: DIODE, Diode_SMD:D_1206_3216Metric, B.Cu at (104.8, 138.4)
- added ENTER1: SW_Push, Button_Switch_Keyboard:SW_Cherry_MX1A_2.25u_PCB, F.Cu at (341.6, 128.3)
- added ESC1: SW_Push, Button_Switch_Keyboard:SW_Cherry_MX1A_1.00u_PCB, F.Cu at (71.1, 87.6)
- added FN1: SW_Push, Button_Switch_Keyboard:SW_Cherry_MX1A_1.75u_PCB, F.Cu at (78.2, 128.3)
- added G***: LOGO, Graphics:pig, B.Cu at (82.8, 167.1)
- added MINI_USB_B: USB_B_Mini, Connector_USB:USB_Mini-B_Lumberg_2486_01_Horizontal, B.Cu at (322.6, 86.4)
- added N0: SW_Push, Button_Switch_Keyboard:SW_Cherry_MX1A_1.00u_PCB, F.Cu at (274.3, 87.6)
- added N1: SW_Push, Button_Switch_Keyboard:SW_Cherry_MX1A_1.00u_PCB, F.Cu at (91.4, 87.6)
- added N2: SW_Push, Button_Switch_Keyboard:SW_Cherry_MX1A_1.00u_PCB, F.Cu at (111.8, 87.6)
- added N3: SW_Push, Button_Switch_Keyboard:SW_Cherry_MX1A_1.00u_PCB, F.Cu at (132.1, 87.6)
- added N4: SW_Push, Button_Switch_Keyboard:SW_Cherry_MX1A_1.00u_PCB, F.Cu at (152.4, 87.6)
- added N5: SW_Push, Button_Switch_Keyboard:SW_Cherry_MX1A_1.00u_PCB, F.Cu at (172.7, 87.6)
- added N6: SW_Push, Button_Switch_Keyboard:SW_Cherry_MX1A_1.00u_PCB, F.Cu at (193.0, 87.6)
- added N7: SW_Push, Button_Switch_Keyboard:SW_Cherry_MX1A_1.00u_PCB, F.Cu at (213.4, 87.6)
- added N8: SW_Push, Button_Switch_Keyboard:SW_Cherry_MX1A_1.00u_PCB, F.Cu at (233.7, 87.6)
- added N9: SW_Push, Button_Switch_Keyboard:SW_Cherry_MX1A_1.00u_PCB, F.Cu at (254.0, 87.6)
- added R2: 22, Resistor_SMD:R_2010_5025Metric_Pad1.52x2.65mm_HandSolder, B.Cu at (223.5, 177.8)
- added R3: 10k, Resistor_SMD:R_2010_5025Metric_Pad1.52x2.65mm_HandSolder, B.Cu at (233.7, 177.8)
- added R4: 330, Resistor_SMD:R_2010_5025Metric_Pad1.52x2.65mm_HandSolder, B.Cu at (224.7, 171.7)
- added R5: 330, Resistor_SMD:R_2010_5025Metric_Pad1.52x2.65mm_HandSolder, B.Cu at (224.7, 167.9)
- added R6: 330, Resistor_SMD:R_2010_5025Metric_Pad1.52x2.65mm_HandSolder, B.Cu at (224.7, 164.1)
- added R7: 10k, Resistor_SMD:R_2010_5025Metric_Pad1.52x2.65mm_HandSolder, B.Cu at (218.4, 177.8)
- added SHIFT_LEFT1: SW_Push, Button_Switch_Keyboard:SW_Cherry_MX1A_2.25u_PCB, F.Cu at (83.1, 148.3)
- added SHIFT_RIGHT1: SW_Push, Button_Switch_Keyboard:SW_Cherry_MX1A_1.75u_PCB, F.Cu at (346.7, 148.6)
- added SPACE1: SW_Push, Button_Switch_Keyboard:SW_Cherry_MX1A_6.25u_PCB, F.Cu at (196.8, 168.9)
- added SUPER1: SW_Push, Button_Switch_Keyboard:SW_Cherry_MX1A_1.25u_PCB, F.Cu at (99.1, 168.9)
- added TAB1: SW_Push, Button_Switch_Keyboard:SW_Cherry_MX1A_1.50u_PCB, F.Cu at (75.9, 108.0)
- added U1: ATmega32U4-AU, Package_QFP:TQFP-44_10x10mm_P0.8mm, B.Cu at (164.5, 168.9)
- added Y1: Crystal, Crystal:Crystal_SMD_5032-2Pin_5.0x3.2mm_HandSoldering, B.Cu at (164.5, 180.6)
- added [1: SW_Push, Button_Switch_Keyboard:SW_Cherry_MX1A_1.00u_PCB, F.Cu at (304.2, 108.0)
- added \1: SW_Push, Button_Switch_Keyboard:SW_Cherry_MX1A_1.50u_PCB, F.Cu at (349.2, 108.0)
- added ]1: SW_Push, Button_Switch_Keyboard:SW_Cherry_MX1A_1.00u_PCB, F.Cu at (324.5, 108.0)
- added a1: SW_Push, Button_Switch_Keyboard:SW_Cherry_MX1A_1.00u_PCB, F.Cu at (106.0, 128.3)
- added b1: SW_Push, Button_Switch_Keyboard:SW_Cherry_MX1A_1.00u_PCB, F.Cu at (196.8, 148.6)
- added c1: SW_Push, Button_Switch_Keyboard:SW_Cherry_MX1A_1.00u_PCB, F.Cu at (156.2, 148.6)
- added d1: SW_Push, Button_Switch_Keyboard:SW_Cherry_MX1A_1.00u_PCB, F.Cu at (146.7, 128.3)
- added e1: SW_Push, Button_Switch_Keyboard:SW_Cherry_MX1A_1.00u_PCB, F.Cu at (141.6, 108.0)
- added f1: SW_Push, Button_Switch_Keyboard:SW_Cherry_MX1A_1.00u_PCB, F.Cu at (167.0, 128.3)
- added g1: SW_Push, Button_Switch_Keyboard:SW_Cherry_MX1A_1.00u_PCB, F.Cu at (187.2, 128.3)
- added h1: SW_Push, Button_Switch_Keyboard:SW_Cherry_MX1A_1.00u_PCB, F.Cu at (207.6, 128.3)
- added i1: SW_Push, Button_Switch_Keyboard:SW_Cherry_MX1A_1.00u_PCB, F.Cu at (243.2, 108.0)
- added j1: SW_Push, Button_Switch_Keyboard:SW_Cherry_MX1A_1.00u_PCB, F.Cu at (228.0, 128.3)
- added k1: SW_Push, Button_Switch_Keyboard:SW_Cherry_MX1A_1.00u_PCB, F.Cu at (248.3, 128.3)
- added l1: SW_Push, Button_Switch_Keyboard:SW_Cherry_MX1A_1.00u_PCB, F.Cu at (268.6, 128.3)
- added m1: SW_Push, Button_Switch_Keyboard:SW_Cherry_MX1A_1.00u_PCB, F.Cu at (237.5, 148.6)
- added n1: SW_Push, Button_Switch_Keyboard:SW_Cherry_MX1A_1.00u_PCB, F.Cu at (217.2, 148.6)
- added o1: SW_Push, Button_Switch_Keyboard:SW_Cherry_MX1A_1.00u_PCB, F.Cu at (263.5, 108.0)
- added p1: SW_Push, Button_Switch_Keyboard:SW_Cherry_MX1A_1.00u_PCB, F.Cu at (283.8, 108.0)
- added q1: SW_Push, Button_Switch_Keyboard:SW_Cherry_MX1A_1.00u_PCB, F.Cu at (101.0, 108.0)
- added r1: SW_Push, Button_Switch_Keyboard:SW_Cherry_MX1A_1.00u_PCB, F.Cu at (161.9, 108.0)
- added s1: SW_Push, Button_Switch_Keyboard:SW_Cherry_MX1A_1.00u_PCB, F.Cu at (126.4, 128.3)
- added t1: SW_Push, Button_Switch_Keyboard:SW_Cherry_MX1A_1.00u_PCB, F.Cu at (182.2, 108.0)
- added u1: SW_Push, Button_Switch_Keyboard:SW_Cherry_MX1A_1.00u_PCB, F.Cu at (222.9, 108.0)
- added v1: SW_Push, Button_Switch_Keyboard:SW_Cherry_MX1A_1.00u_PCB, F.Cu at (176.5, 148.6)
- added w1: SW_Push, Button_Switch_Keyboard:SW_Cherry_MX1A_1.00u_PCB, F.Cu at (121.3, 108.0)
- added x1: SW_Push, Button_Switch_Keyboard:SW_Cherry_MX1A_1.00u_PCB, F.Cu at (135.9, 148.6)
- added y1: SW_Push, Button_Switch_Keyboard:SW_Cherry_MX1A_1.00u_PCB, F.Cu at (202.6, 108.0)
- added z1: SW_Push, Button_Switch_Keyboard:SW_Cherry_MX1A_1.00u_PCB, F.Cu at (115.6, 148.6)
- D1: value LED -> LED_CRGB; footprint LED_THT:LED_Rectangular_W5.0mm_H2.0mm_Horizontal_O1.27mm_Z1.0mm -> LED_THT:LED_D5.0mm-4_RGB
- R1: value R -> 22; footprint Resistor_THT:R_Axial_DIN0207_L6.3mm_D2.5mm_P2.54mm_Vertical -> Resistor_SMD:R_2010_5025Metric_Pad1.52x2.65mm_HandSolder; moved to B.Cu
- SW1: footprint Button_Switch_Keyboard:SW_Cherry_MX1A_1.00u_PCB -> Button_Switch_THT:SW_PUSH_6mm; moved to B.Cu
- moved D1 290.9 mm to (350.5, 171.4), turned to 270 degrees
- moved SW1 215.3 mm to (254.0, 171.4), turned to 180 degrees
- moved R1 179.6 mm to (228.6, 177.8), turned to 270 degrees
Connections:
- D1 pad 1: Net-(BT1-Pad2) -> /GND
- R1 pad 1: Net-(D1-Pad2) -> Net-(R1-Pad1)
- R1 pad 2: Net-(R1-Pad2) -> Net-(J1-Pad3)
- SW1 pad 1: Net-(BT1-Pad1) -> /GND
- SW1 pad 2: Net-(R1-Pad2) -> Net-(R3-Pad2)
Routing:
- net Net-(J1-Pad2): track 0.00 -> 285.4 mm
- net Net-(J1-Pad3): track 0.00 -> 284.6 mm
- net /VCC: track 0.00 -> 274.3 mm
- net /col0: track 0.00 -> 200.5 mm
- net Net-(D1-Pad4): track 0.00 -> 130.4 mm
- net Net-(D1-Pad3): track 0.00 -> 128.8 mm
- net Net-(D1-Pad2): track 17.6 -> 127.1 mm
- net Net-(R1-Pad1): track 0.00 -> 72.0 mm, vias 0 -> 2
- net Net-(R7-Pad2): track 0.00 -> 69.3 mm
- net Net-(R2-Pad1): track 0.00 -> 68.1 mm, vias 0 -> 2
- net Net-(BT1-Pad1): track 64.7 -> 0.00 mm
- net Net-(BT1-Pad2): track 63.9 -> 0.00 mm
- net /LED_G: track 0.00 -> 61.4 mm
- net Net-(C2-Pad1): track 0.00 -> 60.8 mm
- net /LED_B: track 0.00 -> 60.6 mm
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- added copper zone on B.Cu, net /GND
- added copper zone on F.Cu, net /GND
Other:
- board size 88.9 x 41.9 mm -> 304.8 x 103.5 mm

Commit message: almost finished routing
Routing:
- net /ROW1: track 0.00 -> 302.9 mm
- net /ROW0: track 0.00 -> 292.9 mm
- net /ROW2: track 0.00 -> 288.3 mm
- net /ROW3: track 0.00 -> 237.5 mm
- net /col0: track 200.5 -> 90.1 mm
- net /col12: track 0.00 -> 104.9 mm
- net /col2: track 0.00 -> 95.5 mm
- net /col10: track 0.00 -> 95.5 mm
- net /col11: track 0.00 -> 94.4 mm
- net /col13: track 0.00 -> 93.6 mm
- net /col6: track 0.00 -> 91.8 mm
- net /col7: track 0.00 -> 71.5 mm
- net /col3: track 0.00 -> 71.5 mm
- net /col8: track 0.00 -> 71.5 mm
- net /col9: track 0.00 -> 71.5 mm
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
Commit message: finish pcb
Parts:
- added MOUNT1: MountingHole_2.5mm, MountingHole:MountingHole_2.5mm, B.Cu at (357.0, 91.0)
- added MOUNT2: MountingHole_2.5mm, MountingHole:MountingHole_2.5mm, B.Cu at (357.0, 179.0)
- added MOUNT3: MountingHole_2.5mm, MountingHole:MountingHole_2.5mm, B.Cu at (204.0, 175.0)
- added MOUNT4: MountingHole_2.5mm, MountingHole:MountingHole_2.5mm, B.Cu at (84.0, 178.0)
- added MOUNT5: MountingHole_2.5mm, MountingHole:MountingHole_2.5mm, B.Cu at (61.5, 105.9)
- added MOUNT6: MountingHole_2.5mm, MountingHole:MountingHole_2.5mm, B.Cu at (221.0, 85.0)
- added MOUNT7: MountingHole_2.5mm, MountingHole:MountingHole_2.5mm, B.Cu at (195.0, 133.0)
- D10, D11, D12, D13, D14, D15, D16, D17, D18, D19, D2, D20, D21, D22, D23, D24, D25, D26, D27, D28, D29, D3, D30, D31, D32, D33, D34, D35, D36, D37, D38, D39, D4, D40, D41, D42, D43, D44, D45, D46, D47, D48, D49, D5, D50, D51, D52, D53, D54, D55, D56, D57, D58, D59, D6, D60, D61, D62, D63, D7, D8, D9: footprint Diode_SMD:D_1206_3216Metric -> Diode_SMD:D_1206_3216Metric_Pad1.42x1.75mm_HandSolder
- moved G*** 0.89 mm to (83.0, 168.0)
Routing:
- net /ROW4: track 0.00 -> 304.6 mm, vias 0 -> 4
- net /col13: track 93.6 -> 261.2 mm, vias 0 -> 3
- net /col12: track 104.9 -> 270.0 mm, vias 0 -> 7
- net /VCC: track 274.3 -> 437.4 mm, vias 0 -> 13
- net /col11: track 94.4 -> 243.6 mm, vias 0 -> 3
- net /col10: track 95.5 -> 223.8 mm, vias 0 -> 5
- net /col9: track 71.5 -> 189.5 mm, vias 0 -> 3
- net /col0: track 90.1 -> 204.4 mm, vias 0 -> 1
- net /col8: track 71.5 -> 162.9 mm, vias 0 -> 1
- net /col1: track 90.2 -> 177.3 mm, vias 0 -> 1
- net Net-(R3-Pad2): track 22.1 -> 107.9 mm, vias 2 -> 8
- net /ROW0: track 292.9 -> 376.1 mm, vias 0 -> 2
- net /GND: track 0.00 -> 82.9 mm, vias 0 -> 8
- net /ROW3: track 237.5 -> 314.2 mm, vias 0 -> 2
- net /col7: track 71.5 -> 143.9 mm, vias 0 -> 1
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Other:
- board text added: "Jacob's keyboard, REV 1"

Commit message: save
Parts:
- removed D1: LED_CRGB, LED_THT:LED_D5.0mm-4_RGB
- removed the G*** at (83.0, 168.0)
- removed MINI_USB_B: USB_B_Mini, Connector_USB:USB_Mini-B_Lumberg_2486_01_Horizontal
- removed MOUNT6, MOUNT7: MountingHole_2.5mm, MountingHole:MountingHole_2.5mm
- removed SW1: SW_Push, Button_Switch_THT:SW_PUSH_6mm
- added G***: LOGO, Graphics:space, F.Cu at (174.0, 148.8)
- added G***: LOGO, Graphics:space3, F.Cu at (246.1, 52.3)
- added G***: LOGO, Graphics:brain, F.Cu at (137.5, 51.3)
- added J1: USB_B_Micro, Connector_USB:USB_Micro-B_Molex_47346-0001, F.Cu at (60.7, 46.2)
- added RESET: SW_Push, Button_Switch_THT:SW_PUSH_6mm_H4.3mm, F.Cu at (171.4, 48.1)
- added RGB1: LED_CRGB, LED_THT:LED_D5.0mm-4_RGB, F.Cu at (317.8, 51.3)
- ALT_RIGHT1: footprint Button_Switch_Keyboard:SW_Cherry_MX1A_1.25u_PCB -> Button_Switch_Keyboard:SW_Cherry_MX1A_1.50u_PCB
- C1, C2, C3: footprint Capacitor_SMD:C_1812_4532Metric_Pad1.30x3.40mm_HandSolder -> Capacitor_SMD:C_1206_3216Metric_Pad1.42x1.75mm_HandSolder; moved to F.Cu
- D10, D11, D12, D13, D14, D15, D16, D17, D18, D19, D2, D20, D21, D22, D23, D24, D25, D26, D27, D28, D29, D3, D30, D31, D32, D33, D34, D35, D36, D37, D38, D39, D4, D40, D41, D42, D43, D44, D45, D46, D47, D48, D49, D5, D50, D51, D52, D53, D54, D55, D56, D57, D58, D59, D6, D60, D61, D62, D63, D7, D8, D9: footprint Diode_SMD:D_1206_3216Metric_Pad1.42x1.75mm_HandSolder -> Diode_SMD:D_SOD-323_HandSoldering
- MOUNT1, MOUNT2, MOUNT3, MOUNT4, MOUNT5, U1: moved to F.Cu
- R1, R2: value 22 -> 330; footprint Resistor_SMD:R_2010_5025Metric_Pad1.52x2.65mm_HandSolder -> Resistor_THT:R_Axial_DIN0207_L6.3mm_D2.5mm_P7.62mm_Horizontal; moved to F.Cu
- R3: value 10k -> 330; footprint Resistor_SMD:R_2010_5025Metric_Pad1.52x2.65mm_HandSolder -> Resistor_THT:R_Axial_DIN0207_L6.3mm_D2.5mm_P7.62mm_Horizontal; moved to F.Cu
- R4, R5: value 330 -> 22; footprint Resistor_SMD:R_2010_5025Metric_Pad1.52x2.65mm_HandSolder -> Resistor_THT:R_Axial_DIN0207_L6.3mm_D2.5mm_P7.62mm_Horizontal; moved to F.Cu
- R6: value 330 -> 10k; footprint Resistor_SMD:R_2010_5025Metric_Pad1.52x2.65mm_HandSolder -> Resistor_THT:R_Axial_DIN0207_L6.3mm_D2.5mm_P7.62mm_Horizontal; moved to F.Cu
- R7: footprint Resistor_SMD:R_2010_5025Metric_Pad1.52x2.65mm_HandSolder -> Resistor_THT:R_Axial_DIN0207_L6.3mm_D2.5mm_P7.62mm_Horizontal; moved to F.Cu
- Y1: value Crystal -> Crystal_GND2; footprint Crystal:Crystal_SMD_5032-2Pin_5.0x3.2mm_HandSoldering -> Crystal:Crystal_SMD_3225-4Pin_3.2x2.5mm_HandSoldering; moved to F.Cu
- moved MOUNT3 205.2 mm to (41.8, 49.3)
- moved R5 190.6 mm to (77.8, 46.4)
- moved R4 190.5 mm to (77.8, 50.5)
- moved C2 185.5 mm to (73.9, 54.1), turned to 180 degrees
- moved R3 158.3 mm to (321.6, 46.1), turned to 180 degrees
- moved R2 157.0 mm to (324.5, 57.5), turned to 90 degrees
- moved R7 154.9 mm to (123.8, 55.1), turned to 90 degrees
- moved R1 145.6 mm to (310.9, 57.7), turned to 90 degrees
- moved MOUNT2 132.7 mm to (332.7, 48.6)
- moved C1 130.6 mm to (147.9, 48.7), turned to 0 degrees
- moved Y1 129.2 mm to (151.7, 52.0), turned to 45 degrees
- moved R6 125.8 mm to (161.8, 55.1), turned to 90 degrees
- moved C3 125.5 mm to (147.6, 56.1), turned to 180 degrees
- moved U1 120.5 mm to (137.5, 51.5), turned to 90 degrees
- moved MOUNT5 115.0 mm to (176.3, 98.8)
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Connections:
- C1 pad 1: /GND -> GND
- C2 pad 2: /GND -> GND
- C3 pad 1: /GND -> GND
- R1 pad 2: Net-(J1-Pad3) -> /LED_B
- R2 pad 2: Net-(J1-Pad2) -> /LED_G
- R3 pad 1: /VCC -> Net-(R3-Pad1)
- R3 pad 2: Net-(R3-Pad2) -> /LED_R
- R4 pad 1: Net-(D1-Pad4) -> Net-(R4-Pad1)
- R4 pad 2: /LED_B -> Net-(J1-Pad3)
- R5 pad 1: Net-(D1-Pad3) -> Net-(R5-Pad1)
- R5 pad 2: /LED_G -> Net-(J1-Pad2)
- R6 pad 1: Net-(D1-Pad2) -> VCC
- R6 pad 2: /LED_R -> Net-(R6-Pad2)
- R7 pad 1: /GND -> GND
- U1 pad 13: Net-(R3-Pad2) -> Net-(R6-Pad2)
- U1 pad 14: /VCC -> VCC
- U1 pad 15: /GND -> GND
- U1 pad 2: /VCC -> VCC
- U1 pad 23: /GND -> GND
- U1 pad 24: /VCC -> VCC
- U1 pad 3: Net-(R2-Pad1) -> Net-(R5-Pad1)
- U1 pad 34: /VCC -> VCC
- U1 pad 35: /GND -> GND
- U1 pad 4: Net-(R1-Pad1) -> Net-(R4-Pad1)
- U1 pad 43: /GND -> GND
- U1 pad 44: /VCC -> VCC
- U1 pad 5: /GND -> GND
- U1 pad 7: /VCC -> VCC
- Y1 pad 1: Net-(C1-Pad2) -> Net-(C3-Pad2)
- Y1 pad 2: Net-(C3-Pad2) -> GND
Routing:
- net /VCC: track 437.4 -> 0.00 mm, vias 13 -> 0
- net Net-(J1-Pad2): track 285.4 -> 12.0 mm
- net Net-(J1-Pad3): track 283.8 -> 11.3 mm
- net /ROW4: track 304.6 -> 491.2 mm, vias 4 -> 1
- net /LED_G: track 61.4 -> 223.7 mm, vias 0 -> 1
- net /LED_R: track 60.2 -> 206.7 mm
- net /LED_B: track 62.4 -> 201.1 mm, vias 0 -> 1
- net Net-(D1-Pad4): track 130.4 -> 0.00 mm
- net Net-(D1-Pad3): track 128.8 -> 0.00 mm
- net Net-(D1-Pad2): track 127.1 -> 0.00 mm
- net Net-(R3-Pad2): track 107.9 -> 0.00 mm, vias 8 -> 0
- net VCC: track 0.00 -> 83.6 mm, vias 0 -> 8
- net /GND: track 82.9 -> 0.00 mm, vias 8 -> 0
- net /ROW0: track 376.1 -> 300.0 mm, vias 2 -> 1
- net GND: track 0.00 -> 73.2 mm, vias 0 -> 7
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- added copper zone on F.Cu, net GND
- added copper zone on B.Cu, net VCC
- removed copper zone on B.Cu, net /GND
- removed copper zone on F.Cu, net /GND
Other:
- board size 304.8 x 103.5 mm -> 299.5 x 116.8 mm
- rule pad_to_mask_clearance: 0.2 -> 0
- board text added: "Jacob Garby Keyboard REV 2 FEB 19"
- board text removed: "Jacob's keyboard, REV 1"

Commit message: check
Parts:
- removed '1, ,1, -1, .1, /1, ;1, =1, ARROW_DOWN1, ARROW_LEFT1, ARROW_RIGHT1, ARROW_UP1, ESC1, N0, N1, N2, N3, N4, N5, N6, N7, N8, N9, [1, ]1, a1, b1, c1, d1, e1, f1, g1, h1, i1, j1, k1, l1, m1, n1, o1, p1, q1, r1, s1, t1, u1, v1, w1, x1, y1, z1: SW_Push, Button_Switch_Keyboard:SW_Cherry_MX1A_1.00u_PCB
- removed ALT_LEFT1, CTRL1, SUPER1: SW_Push, Button_Switch_Keyboard:SW_Cherry_MX1A_1.25u_PCB
- removed ALT_RIGHT1, TAB1, \1: SW_Push, Button_Switch_Keyboard:SW_Cherry_MX1A_1.50u_PCB
- removed BACKSPACE1: SW_Push, Button_Switch_Keyboard:SW_Cherry_MX1A_2.00u_PCB
- removed ENTER1, SHIFT_LEFT1: SW_Push, Button_Switch_Keyboard:SW_Cherry_MX1A_2.25u_PCB
- removed FN1, SHIFT_RIGHT1: SW_Push, Button_Switch_Keyboard:SW_Cherry_MX1A_1.75u_PCB
- removed G***: LOGO, Graphics:space
- removed G***: LOGO, Graphics:space3
- removed G***: LOGO, Graphics:brain
- removed MOUNT1, MOUNT2, MOUNT3, MOUNT4, MOUNT5: MountingHole_2.5mm, MountingHole:MountingHole_2.5mm
- removed RESET: SW_Push, Button_Switch_THT:SW_PUSH_6mm_H4.3mm
- removed RGB1: LED_CRGB, LED_THT:LED_D5.0mm-4_RGB
- removed SPACE1: SW_Push, Button_Switch_Keyboard:SW_Cherry_MX1A_6.25u_PCB
- added C4: 10uF, Capacitor_SMD:C_1206_3216Metric_Pad1.42x1.75mm_HandSolder, F.Cu at (38.6, 30.1)
- added D1: POWER_INDICATOR, LED_THT:LED_D3.0mm, F.Cu at (34.0, 31.3)
- added D64: LED, LED_SMD:LED_1206_3216Metric_Pad1.42x1.75mm_HandSolder, F.Cu at (127.0, 20.9)
- added J2: GND, Connector_Pin:Pin_D1.0mm_L10.0mm_LooseFit, F.Cu at (73.6, 28.7)
- added J3: VCC, Connector_Pin:Pin_D1.0mm_L10.0mm_LooseFit, F.Cu at (49.0, 21.1)
- added J4: SCK, Connector_Pin:Pin_D1.0mm_L10.0mm_LooseFit, F.Cu at (78.0, 28.8)
- added J5: MOSI, Connector_Pin:Pin_D1.0mm_L10.0mm_LooseFit, F.Cu at (104.2, 33.2)
- added J6: MISO, Connector_Pin:Pin_D1.0mm_L10.0mm_LooseFit, F.Cu at (108.4, 33.3)
- added J7: RESET, Connector_Pin:Pin_D1.0mm_L10.0mm_LooseFit, F.Cu at (128.2, 33.9)
- added K0: SW_Push, Button_Switch_Keyboard:SW_Cherry_MX1A_1.00u_PCB, F.Cu at (28.6, 41.6)
- added K1: SW_Push, Button_Switch_Keyboard:SW_Cherry_MX1A_1.00u_PCB, F.Cu at (48.5, 41.6)
- added K10: SW_Push, Button_Switch_Keyboard:SW_Cherry_MX1A_1.00u_PCB, F.Cu at (227.6, 41.6)
- added K11: SW_Push, Button_Switch_Keyboard:SW_Cherry_MX1A_1.00u_PCB, F.Cu at (247.5, 41.6)
- added K12: SW_Push, Button_Switch_Keyboard:SW_Cherry_MX1A_1.00u_PCB, F.Cu at (267.4, 41.6)
- added K13: SW_Push, Button_Switch_Keyboard:SW_Cherry_MX1A_2.00u_PCB, F.Cu at (296.8, 41.6)
- added K14: SW_Push, Button_Switch_Keyboard:SW_Cherry_MX1A_1.50u_PCB, F.Cu at (33.4, 62.1)
- added K15: SW_Push, Button_Switch_Keyboard:SW_Cherry_MX1A_1.00u_PCB, F.Cu at (58.1, 62.1)
- added K16: SW_Push, Button_Switch_Keyboard:SW_Cherry_MX1A_1.00u_PCB, F.Cu at (78.0, 62.1)
- added K17: SW_Push, Button_Switch_Keyboard:SW_Cherry_MX1A_1.00u_PCB, F.Cu at (97.9, 62.1)
- added K18: SW_Push, Button_Switch_Keyboard:SW_Cherry_MX1A_1.00u_PCB, F.Cu at (117.8, 62.1)
- added K19: SW_Push, Button_Switch_Keyboard:SW_Cherry_MX1A_1.00u_PCB, F.Cu at (137.7, 62.1)
- added K2: SW_Push, Button_Switch_Keyboard:SW_Cherry_MX1A_1.00u_PCB, F.Cu at (68.4, 41.6)
- added K20: SW_Push, Button_Switch_Keyboard:SW_Cherry_MX1A_1.00u_PCB, F.Cu at (157.6, 62.1)
- added K21: SW_Push, Button_Switch_Keyboard:SW_Cherry_MX1A_1.00u_PCB, F.Cu at (177.4, 62.1)
- added K22: SW_Push, Button_Switch_Keyboard:SW_Cherry_MX1A_1.00u_PCB, F.Cu at (197.3, 62.1)
- added K23: SW_Push, Button_Switch_Keyboard:SW_Cherry_MX1A_1.00u_PCB, F.Cu at (217.2, 62.1)
- added K24: SW_Push, Button_Switch_Keyboard:SW_Cherry_MX1A_1.00u_PCB, F.Cu at (237.1, 62.1)
- added K25: SW_Push, Button_Switch_Keyboard:SW_Cherry_MX1A_1.00u_PCB, F.Cu at (257.0, 62.1)
- added K26: SW_Push, Button_Switch_Keyboard:SW_Cherry_MX1A_1.00u_PCB, F.Cu at (276.9, 62.1)
- added K27: SW_Push, Button_Switch_Keyboard:SW_Cherry_MX1A_1.50u_PCB, F.Cu at (301.6, 62.1)
- added K28: SW_Push, Button_Switch_Keyboard:SW_Cherry_MX1A_1.75u_PCB, F.Cu at (35.8, 82.5)
- added K29: SW_Push, Button_Switch_Keyboard:SW_Cherry_MX1A_1.00u_PCB, F.Cu at (62.9, 82.5)
- added K3: SW_Push, Button_Switch_Keyboard:SW_Cherry_MX1A_1.00u_PCB, F.Cu at (88.3, 41.6)
- added K30: SW_Push, Button_Switch_Keyboard:SW_Cherry_MX1A_1.00u_PCB, F.Cu at (82.9, 82.5)
- added K31: SW_Push, Button_Switch_Keyboard:SW_Cherry_MX1A_1.00u_PCB, F.Cu at (102.8, 82.5)
- added K32: SW_Push, Button_Switch_Keyboard:SW_Cherry_MX1A_1.00u_PCB, F.Cu at (122.8, 82.5)
- added K33: SW_Push, Button_Switch_Keyboard:SW_Cherry_MX1A_1.00u_PCB, F.Cu at (142.8, 82.5)
- added K34: SW_Push, Button_Switch_Keyboard:SW_Cherry_MX1A_1.00u_PCB, F.Cu at (162.7, 82.5)
- added K35: SW_Push, Button_Switch_Keyboard:SW_Cherry_MX1A_1.00u_PCB, F.Cu at (182.7, 82.5)
- added K36: SW_Push, Button_Switch_Keyboard:SW_Cherry_MX1A_1.00u_PCB, F.Cu at (202.6, 82.5)
- added K37: SW_Push, Button_Switch_Keyboard:SW_Cherry_MX1A_1.00u_PCB, F.Cu at (222.6, 82.5)
- added K38: SW_Push, Button_Switch_Keyboard:SW_Cherry_MX1A_1.00u_PCB, F.Cu at (242.6, 82.5)
- added K39: SW_Push, Button_Switch_Keyboard:SW_Cherry_MX1A_1.00u_PCB, F.Cu at (262.5, 82.5)
- added K4: SW_Push, Button_Switch_Keyboard:SW_Cherry_MX1A_1.00u_PCB, F.Cu at (108.2, 41.6)
- added K40: SW_Push, Button_Switch_Keyboard:SW_Cherry_MX1A_2.25u_PCB, F.Cu at (294.4, 82.5)
- added K41: SW_Push, Button_Switch_Keyboard:SW_Cherry_MX1A_2.25u_PCB, F.Cu at (40.5, 102.9)
- added K42: SW_Push, Button_Switch_Keyboard:SW_Cherry_MX1A_1.00u_PCB, F.Cu at (72.4, 102.9)
- added K43: SW_Push, Button_Switch_Keyboard:SW_Cherry_MX1A_1.00u_PCB, F.Cu at (92.3, 103.0)
- added K44: SW_Push, Button_Switch_Keyboard:SW_Cherry_MX1A_1.00u_PCB, F.Cu at (112.3, 103.0)
- added K45: SW_Push, Button_Switch_Keyboard:SW_Cherry_MX1A_1.00u_PCB, F.Cu at (132.3, 103.0)
- added K46: SW_Push, Button_Switch_Keyboard:SW_Cherry_MX1A_1.00u_PCB, F.Cu at (152.3, 103.0)
- added K47: SW_Push, Button_Switch_Keyboard:SW_Cherry_MX1A_1.00u_PCB, F.Cu at (172.2, 103.0)
- added K48: SW_Push, Button_Switch_Keyboard:SW_Cherry_MX1A_1.00u_PCB, F.Cu at (192.2, 103.0)
- added K49: SW_Push, Button_Switch_Keyboard:SW_Cherry_MX1A_1.00u_PCB, F.Cu at (212.2, 103.0)
- added K5: SW_Push, Button_Switch_Keyboard:SW_Cherry_MX1A_1.00u_PCB, F.Cu at (128.1, 41.6)
- added K50: SW_Push, Button_Switch_Keyboard:SW_Cherry_MX1A_1.00u_PCB, F.Cu at (232.1, 103.0)
- added K51: SW_Push, Button_Switch_Keyboard:SW_Cherry_MX1A_1.00u_PCB, F.Cu at (252.1, 103.0)
- added K52: SW_Push, Button_Switch_Keyboard:SW_Cherry_MX1A_1.00u_PCB, F.Cu at (272.1, 103.0)
- added K53: SW_Push, Button_Switch_Keyboard:SW_Cherry_MX1A_1.75u_PCB, F.Cu at (299.2, 103.0)
- added K54: SW_Push, Button_Switch_Keyboard:SW_Cherry_MX1A_1.25u_PCB, F.Cu at (31.0, 123.3)
- added K55: SW_Push, Button_Switch_Keyboard:SW_Cherry_MX1A_1.25u_PCB, F.Cu at (56.1, 123.3)
- added K56: SW_Push, Button_Switch_Keyboard:SW_Cherry_MX1A_1.25u_PCB, F.Cu at (81.3, 123.3)
- added K57: SW_Push, Button_Switch_Keyboard:SW_Cherry_MX1A_6.25u_PCB, F.Cu at (154.0, 123.3)
- added K58: SW_Push, Button_Switch_Keyboard:SW_Cherry_MX1A_1.25u_PCB, F.Cu at (226.8, 123.3)
- added K59: SW_Push, Button_Switch_Keyboard:SW_Cherry_MX1A_1.00u_PCB, F.Cu at (252.2, 123.3)
- added K6: SW_Push, Button_Switch_Keyboard:SW_Cherry_MX1A_1.00u_PCB, F.Cu at (148.0, 41.6)
- added K60: SW_Push, Button_Switch_Keyboard:SW_Cherry_MX1A_1.00u_PCB, F.Cu at (272.1, 123.3)
- added K61: SW_Push, Button_Switch_Keyboard:SW_Cherry_MX1A_1.00u_PCB, F.Cu at (292.0, 123.3)
- added K7: SW_Push, Button_Switch_Keyboard:SW_Cherry_MX1A_1.00u_PCB, F.Cu at (167.9, 41.6)
- added K8: SW_Push, Button_Switch_Keyboard:SW_Cherry_MX1A_1.00u_PCB, F.Cu at (187.8, 41.6)
- added K9: SW_Push, Button_Switch_Keyboard:SW_Cherry_MX1A_1.00u_PCB, F.Cu at (207.7, 41.6)
- added R10: 1k, Resistor_SMD:R_1206_3216Metric, F.Cu at (177.4, 21.5)
- added R8: 300, Resistor_SMD:R_1206_3216Metric, F.Cu at (30.8, 25.7)
- added R9: 1k, Resistor_SMD:R_1206_3216Metric, F.Cu at (177.4, 24.8)
- added REF**: MountingHole_2.5mm_Pad, MountingHole:MountingHole_2.5mm_Pad, F.Cu at (21.8, 33.3)
- added REF**: MountingHole_2.5mm_Pad, MountingHole:MountingHole_2.5mm_Pad, F.Cu at (21.8, 21.9)
- added REF**: MountingHole_2.5mm_Pad, MountingHole:MountingHole_2.5mm_Pad, F.Cu at (307.6, 33.3)
- added REF**: MountingHole_2.5mm_Pad, MountingHole:MountingHole_2.5mm_Pad, F.Cu at (166.6, 27.5)
- added REF**: MountingHole_2.5mm_Pad, MountingHole:MountingHole_2.5mm_Pad, F.Cu at (85.5, 77.5)
- added REF**: MountingHole_2.5mm_Pad, MountingHole:MountingHole_2.5mm_Pad, F.Cu at (204.8, 77.2)
- added REF**: MountingHole_2.5mm_Pad, MountingHole:MountingHole_2.5mm_Pad, F.Cu at (137.2, 128.0)
- added REF**: MountingHole_2.5mm_Pad, MountingHole:MountingHole_2.5mm_Pad, F.Cu at (41.0, 128.3)
- added REF**: MountingHole_2.5mm_Pad, MountingHole:MountingHole_2.5mm_Pad, F.Cu at (307.6, 132.9)
- added REF**: MountingHole_2.5mm_Pad, MountingHole:MountingHole_2.5mm_Pad, F.Cu at (307.6, 21.9)
- added SW1: RESET, Button_Switch_THT:SW_PUSH_6mm_H4.3mm, F.Cu at (69.4, 30.3)
- added SW2: SW_DIP_x04, Button_Switch_THT:SW_DIP_SPSTx04_Slide_6.7x11.72mm_W7.62mm_P2.54mm_LowProfile, F.Cu at (182.2, 22.5)
- C1, C3, Y1: moved to B.Cu
- J1: value USB_B_Micro -> USB_B_Mini; footprint Connector_USB:USB_Micro-B_Molex_47346-0001 -> keyboard:Molex_OTG_54819_Right_angle
- R1, R4, R5, R6, R7: footprint Resistor_THT:R_Axial_DIN0207_L6.3mm_D2.5mm_P7.62mm_Horizontal -> Resistor_SMD:R_1206_3216Metric
- R2, R3: value 330 -> 1k; footprint Resistor_THT:R_Axial_DIN0207_L6.3mm_D2.5mm_P7.62mm_Horizontal -> Resistor_SMD:R_1206_3216Metric
- moved R1 181.7 mm to (133.0, 20.9), turned to 0 degrees
- moved R2 149.4 mm to (177.4, 31.5), turned to 180 degrees
- moved R3 145.3 mm to (177.4, 28.2)
- moved R6 114.2 mm to (51.6, 25.1), turned to 0 degrees
- moved R7 42.6 mm to (154.5, 25.5), turned to 135 degrees
- moved R4 32.9 mm to (51.6, 30.7)
- moved R5 32.1 mm to (51.6, 27.9)
- moved C2 30.2 mm to (51.8, 33.5)
- moved D56 29.6 mm to (277.4, 71.9), turned to 0 degrees
- moved D57 29.4 mm to (294.8, 92.3), turned to 0 degrees
- moved D49 29.1 mm to (224.8, 132.9), turned to 0 degrees
- moved D46 29.1 mm to (237.8, 71.9), turned to 0 degrees
- moved D41 29.0 mm to (208.6, 51.5), turned to 0 degrees
- moved D45 29.0 mm to (228.4, 51.5), turned to 0 degrees
- moved D60 28.9 mm to (297.8, 51.5), turned to 0 degrees
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Connections:
- net /LED_B renamed /LED
- net Net-(R6-Pad2) renamed /RST
- R2 pad 1: Net-(R2-Pad1) -> /DIP4
- R2 pad 2: /LED_G -> VCC
- R3 pad 1: Net-(R3-Pad1) -> /DIP3
- R3 pad 2: /LED_R -> VCC
- U1 pad 1: /col13 -> /col0
- U1 pad 10: /ROW2 -> /col3
- U1 pad 11: /ROW3 -> /col4
- U1 pad 12: /col2 -> /col5
- U1 pad 18: /col5 -> /col6
- U1 pad 19: /col6 -> /col7
- U1 pad 20: /col7 -> /col8
- U1 pad 21: /col8 -> /col9
- U1 pad 25: /col9 -> /col11
- U1 pad 26: /col11 -> /col12
- U1 pad 27: /col12 -> /col13
- U1 pad 28: /ROW4 -> /ROW0
- U1 pad 29: /col0 -> /ROW1
- U1 pad 30: /col1 -> /ROW2
- U1 pad 31: /col3 -> /ROW3
- U1 pad 32: /col4 -> /ROW4
- U1 pad 37: Net-(U1-Pad37) -> /DIP4
- U1 pad 38: Net-(U1-Pad38) -> /DIP3
- U1 pad 39: /LED_R -> /DIP2
- U1 pad 40: /LED_G -> /DIP1
- U1 pad 8: /ROW0 -> /col1
- U1 pad 9: /ROW1 -> /col2
Routing:
- net VCC: track 83.6 -> 309.6 mm, vias 8 -> 2
- net /LED_G: track 223.7 -> 0.00 mm, vias 1 -> 0
- net /LED_R: track 206.7 -> 0.00 mm
- net /LED: track 201.1 -> 11.1 mm, vias 1 -> 0
- net /ROW2: track 332.2 -> 494.9 mm, vias 3 -> 1
- net /ROW1: track 320.5 -> 480.1 mm, vias 3 -> 1
- net /ROW3: track 355.0 -> 513.6 mm, vias 3 -> 1
- net /ROW0: track 300.0 -> 457.6 mm
- net GND: track 73.2 -> 12.1 mm, vias 7 -> 0
- net /RST: track 36.5 -> 95.2 mm
- net /col12: track 277.1 -> 221.6 mm, vias 1 -> 0
- net /col13: track 285.3 -> 237.3 mm, vias 2 -> 0
- net /ROW4: track 491.2 -> 536.9 mm
- net /DIP4: track 0.00 -> 45.2 mm
- net /DIP3: track 0.00 -> 43.6 mm
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- added copper zone on B.Cu, net GND
- removed copper zone on B.Cu, net VCC
Other:
- board size 299.5 x 116.8 mm -> 298 x 120.6 mm
- board text removed: "Jacob Garby Keyboard REV 2 FEB 19"

Commit message: update
Parts:
- added REF**: OSHW-Logo_11.4x12mm_SilkScreen, Symbol:OSHW-Logo_11.4x12mm_SilkScreen, B.Cu at (283.2, 106.4)
- added TP1: TestPoint_Probe, TestPoint:TestPoint_Pad_D1.0mm, B.Cu at (134.6, 34.8)
- added TP2: TestPoint_Probe, TestPoint:TestPoint_Pad_D1.0mm, F.Cu at (42.2, 30.8)
- added TP3: TestPoint_Probe, TestPoint:TestPoint_Pad_D1.0mm, F.Cu at (22.0, 26.8)
- D1: value POWER_INDICATOR -> PWR; footprint LED_THT:LED_D3.0mm -> LED_SMD:LED_1206_3216Metric_Pad1.42x1.75mm_HandSolder
- SW1: value RESET -> SW_Push
- Y1: value Crystal_GND2 -> 16MHz
- moved R1 106.2 mm to (26.9, 25.4), turned to 90 degrees
- moved D64 100.6 mm to (26.9, 31.4), turned to 90 degrees
- moved J7 52.7 mm to (76.8, 22.2)
- moved C1 13.3 mm to (136.8, 37.5), turned to 0 degrees
- moved J3 13.0 mm to (58.6, 29.8)
- moved C3 12.5 mm to (149.2, 37.2), turned to 180 degrees
- moved J1 9.15 mm to (39.0, 18.2), turned to 0 degrees
- moved D1 3.20 mm to (30.8, 31.4), turned to 90 degrees
- moved R7 1.90 mm to (156.2, 26.2)
- moved Y1 0.59 mm to (142.9, 39.0), turned to 225 degrees
- moved R8 0.30 mm to (30.8, 25.4)
- moved J4 0.05 mm to (78.0, 28.7)
Connections:
- U1 pad 16: Net-(C3-Pad2) -> Net-(C1-Pad2)
- U1 pad 17: Net-(C1-Pad2) -> Net-(C3-Pad2)
Routing:
- net VCC: track 309.6 -> 56.5 mm, vias 2 -> 11
- net /LED: track 11.1 -> 119.6 mm, vias 0 -> 2
- net GND: track 12.1 -> 36.4 mm, vias 0 -> 1
- net /RST: track 95.2 -> 110.4 mm, vias 0 -> 2
- net Net-(D64-Pad2): track 3.11 -> 9.30 mm
- net Net-(C1-Pad2): track 10.2 -> 14.7 mm
- net /col2: track 193.9 -> 191.8 mm
- net Net-(R7-Pad2): track 4.24 -> 6.30 mm
- net Net-(D1-Pad2): track 4.47 -> 3.11 mm
- net Net-(C3-Pad2): track 9.94 -> 8.82 mm
- net Net-(J1-Pad2): track 12.4 -> 11.8 mm
- net Net-(J1-Pad3): track 18.4 -> 17.8 mm
- added copper zone on B.Cu, net VCC
- removed copper zone on B.Cu, net GND
Other:
- outline, holes or cut-outs redrawn
- board text added: "Jacob G Rev. 4"
