File: keyboard1.sch (KiCad schematic (older format))
At the start: 130 parts

Commit message: progress wiring mcu
Parts:
- removed D? (x64): D, symbol Device:D
- removed SW? (x64): SW_Push, symbol Switch:SW_Push
- added C?: CAP, symbol pspice:CAP
- added R? (x2): R22, symbol Device:R
- added SW?: SW_Push, symbol Switch:SW_Push
Connections:
- wire segments 240 -> 29
- no-connect marks 8 -> 1

Commit message: finished wiring up mcu
Parts:
- removed SW?: SW_Push, symbol Switch:SW_Push
- added C1, C3: 22p, symbol pspice:CAP
- added D1: LED_CRGB, symbol Device:LED_CRGB
- added R3, R7: 10k, symbol Device:R
- added R4, R5, R6: 330, symbol Device:R
- added SW1: SW_Push, symbol Switch:SW_Push
- added Y1: Crystal, symbol Device:Crystal
- C2: renamed from C?; value CAP -> 1u
- R1, R2: renamed from R?; value R22 -> 22
- gave numbers to parts that had none: 2
Connections:
- net labels added: GND, LED_B, LED_G, LED_R, ROW0, ROW1, ROW2, ROW3, ROW4, VCC, col0, col1, col10, col11, col12, col13, col2, col3, col4, col5, col6, col7, col8, col9
- wire segments 29 -> 35
- no-connect marks 1 -> 4
Other:
- note added: "This pin going to ground means that the \nRESET pin will activate bootloader mode"
- moved on the sheet: J1, U1

Commit message: finished keyboard schematic
Parts:
- added '1, ,1, -1, .1, /1, ;1, =1, ALT_LEFT1, ALT_RIGHT1, ARROW_DOWN1, ARROW_LEFT1, ARROW_RIGHT1, ARROW_UP1, BACKSPACE1, CTRL1, ENTER1, ESC1, FN1, N0, N1, N2, N3, N4, N5, N6, N7, N8, N9, SHIFT_LEFT1, SHIFT_RIGHT1, SPACE1, SUPER1, TAB1, [1, \1, ]1, a1, b1, c1, d1, e1, f1, g1, h1, i1, j1, k1, l1, m1, n1, o1, p1, q1, r1, s1, t1, u1, v1, w1, x1, y1, z1: SW_Push, symbol Switch:SW_Push
- added D10, D11, D12, D13, D14, D15, D16, D17, D18, D19, D2, D20, D21, D22, D23, D24, D25, D26, D27, D28, D29, D3, D30, D31, D32, D33, D34, D35, D36, D37, D38, D39, D4, D40, D41, D42, D43, D44, D45, D46, D47, D48, D49, D5, D50, D51, D52, D53, D54, D55, D56, D57, D58, D59, D6, D60, D61, D62, D63, D7, D8, D9: DIODE, symbol pspice:DIODE
Connections:
- wire segments 35 -> 220
Other:
- note removed: "This pin going to ground means that the \nRESET pin will activate bootloader mode"
- moved on the sheet: J1, U1

Commit message: pcb progress
Parts:
- '1, ,1, -1, .1, /1, ;1, =1, ARROW_DOWN1, ARROW_LEFT1, ARROW_RIGHT1, ARROW_UP1, ESC1, N0, N1, N2, N3, N4, N5, N6, N7, N8, N9, SW1, [1, ]1, a1, b1, c1, d1, e1, f1, g1, h1, i1, j1, k1, l1, m1, n1, o1, p1, q1, r1, s1, t1, u1, v1, w1, x1, y1, z1: footprint (none) -> Button_Switch_Keyboard:SW_Cherry_MX1A_1.00u_PCB
- ALT_LEFT1, ALT_RIGHT1, CTRL1, SUPER1: footprint (none) -> Button_Switch_Keyboard:SW_Cherry_MX1A_1.25u_PCB
- BACKSPACE1: footprint (none) -> Button_Switch_Keyboard:SW_Cherry_MX1A_2.00u_PCB
- C1, C2, C3: footprint (none) -> Capacitor_THT:C_Disc_D3.0mm_W1.6mm_P2.50mm
- D1: footprint (none) -> LED_THT:LED_D5.0mm-4_RGB
- D10, D11, D12, D13, D14, D15, D16, D17, D18, D19, D2, D20, D21, D22, D23, D24, D25, D26, D27, D28, D29, D3, D30, D31, D32, D33, D34, D35, D36, D37, D38, D39, D4, D40, D41, D42, D43, D44, D45, D46, D47, D48, D49, D5, D50, D51, D52, D53, D54, D55, D56, D57, D58, D59, D6, D60, D61, D62, D63, D7, D8, D9: footprint (none) -> Diode_THT:D_T-1_P5.08mm_Horizontal
- ENTER1, SHIFT_LEFT1: footprint (none) -> Button_Switch_Keyboard:SW_Cherry_MX1A_2.25u_PCB
- FN1, SHIFT_RIGHT1: footprint (none) -> Button_Switch_Keyboard:SW_Cherry_MX1A_1.75u_PCB
- J1: footprint (none) -> Connector_USB:USB_Mini-B_Lumberg_2486_01_Horizontal
- R1, R2, R3, R4, R5, R6, R7: footprint (none) -> Resistor_THT:R_Axial_DIN0204_L3.6mm_D1.6mm_P5.08mm_Horizontal
- SPACE1: footprint (none) -> Button_Switch_Keyboard:SW_Cherry_MX1A_6.25u_PCB
- TAB1, \1: footprint (none) -> Button_Switch_Keyboard:SW_Cherry_MX1A_1.50u_PCB
- Y1: footprint (none) -> Crystal:Crystal_HC49-U_Vertical

Commit message: save
Parts:
- removed C1, C3: 22p, Capacitor_THT:C_Disc_D3.0mm_W1.6mm_P2.50mm, symbol pspice:CAP
- removed C2: 1u, Capacitor_THT:C_Disc_D3.0mm_W1.6mm_P2.50mm, symbol pspice:CAP
- removed J1: USB_B_Mini, Connector_USB:USB_Mini-B_Lumberg_2486_01_Horizontal, symbol Connector:USB_B_Mini
- removed Y1: Crystal, Crystal:Crystal_HC49-U_Vertical, symbol Device:Crystal
- added C1, C3: 22p, Capacitor_SMD:C_1206_3216Metric_Pad1.42x1.75mm_HandSolder, symbol Device:C
- added C2: 1u, Capacitor_SMD:C_1206_3216Metric_Pad1.42x1.75mm_HandSolder, symbol Device:C
- added J1: USB_B_Micro, Connector_USB:USB_Micro-B_Molex_47346-0001, symbol Connector:USB_B_Micro
- added Y1: Crystal_GND2, Crystal:Crystal_SMD_3225-4Pin_3.2x2.5mm_HandSoldering, symbol Device:Crystal_GND2
- D10, D11, D12, D13, D14, D15, D16, D17, D18, D19, D2, D20, D21, D22, D23, D24, D25, D26, D27, D28, D29, D3, D30, D31, D32, D33, D34, D35, D36, D37, D38, D39, D4, D40, D41, D42, D43, D44, D45, D46, D47, D48, D49, D5, D50, D51, D52, D53, D54, D55, D56, D57, D58, D59, D6, D60, D61, D62, D63, D7, D8, D9: footprint Diode_THT:D_T-1_P5.08mm_Horizontal -> Diode_SMD:D_SOD-323_HandSoldering; symbol pspice:DIODE -> Device:D
- R1: renamed from R4; footprint Resistor_THT:R_Axial_DIN0204_L3.6mm_D1.6mm_P5.08mm_Horizontal -> Resistor_THT:R_Axial_DIN0207_L6.3mm_D2.5mm_P7.62mm_Horizontal
- R2: renamed from R5; footprint Resistor_THT:R_Axial_DIN0204_L3.6mm_D1.6mm_P5.08mm_Horizontal -> Resistor_THT:R_Axial_DIN0207_L6.3mm_D2.5mm_P7.62mm_Horizontal
- R3: renamed from R6; footprint Resistor_THT:R_Axial_DIN0204_L3.6mm_D1.6mm_P5.08mm_Horizontal -> Resistor_THT:R_Axial_DIN0207_L6.3mm_D2.5mm_P7.62mm_Horizontal
- R4: renamed from R1; footprint Resistor_THT:R_Axial_DIN0204_L3.6mm_D1.6mm_P5.08mm_Horizontal -> Resistor_THT:R_Axial_DIN0207_L6.3mm_D2.5mm_P7.62mm_Horizontal
- R5: renamed from R2; footprint Resistor_THT:R_Axial_DIN0204_L3.6mm_D1.6mm_P5.08mm_Horizontal -> Resistor_THT:R_Axial_DIN0207_L6.3mm_D2.5mm_P7.62mm_Horizontal
- R6: renamed from R3; footprint Resistor_THT:R_Axial_DIN0204_L3.6mm_D1.6mm_P5.08mm_Horizontal -> Resistor_THT:R_Axial_DIN0207_L6.3mm_D2.5mm_P7.62mm_Horizontal
- R7: footprint Resistor_THT:R_Axial_DIN0204_L3.6mm_D1.6mm_P5.08mm_Horizontal -> Resistor_THT:R_Axial_DIN0207_L6.3mm_D2.5mm_P7.62mm_Horizontal
- SW1: footprint Button_Switch_Keyboard:SW_Cherry_MX1A_1.00u_PCB -> Button_Switch_THT:SW_PUSH_6mm_H4.3mm
- renumbered N0 to N10, D1 to RGB1
Connections:
- wire segments 220 -> 351
- no-connect marks 4 -> 5
Other:
- moved on the sheet: U1

Commit message: check
Parts:
- removed J1: USB_B_Micro, Connector_USB:USB_Micro-B_Molex_47346-0001, symbol Connector:USB_B_Micro
- removed RGB1: LED_CRGB, LED_THT:LED_D5.0mm-4_RGB, symbol Device:LED_CRGB
- added C4: 10uF, Capacitor_SMD:C_1206_3216Metric_Pad1.42x1.75mm_HandSolder, symbol Device:C
- added D1: POWER_INDICATOR, LED_THT:LED_D3.0mm, symbol Device:LED
- added D64: LED, LED_SMD:LED_1806_4516Metric_Pad1.57x1.80mm_HandSolder, symbol Device:LED
- added J1: USB_B_Mini, keyboard:Molex_OTG_54819_Right_angle, symbol Connector:USB_B_Mini
- added J2: GND, Connector_Pin:Pin_D1.0mm_L10.0mm_LooseFit, symbol Connector_Generic:Conn_01x01
- added J3: VCC, Connector_Pin:Pin_D1.0mm_L10.0mm_LooseFit, symbol Connector_Generic:Conn_01x01
- added J4: SCK, Connector_Pin:Pin_D1.0mm_L10.0mm_LooseFit, symbol Connector_Generic:Conn_01x01
- added J5: MOSI, Connector_Pin:Pin_D1.0mm_L10.0mm_LooseFit, symbol Connector_Generic:Conn_01x01
- added J6: MISO, Connector_Pin:Pin_D1.0mm_L10.0mm_LooseFit, symbol Connector_Generic:Conn_01x01
- added J7: RESET, Connector_Pin:Pin_D1.0mm_L10.0mm_LooseFit, symbol Connector_Generic:Conn_01x01
- added R10, R9: 1k, Resistor_SMD:R_1206_3216Metric, symbol Device:R
- added R8: 300, Resistor_SMD:R_1206_3216Metric, symbol Device:R
- added SW2: SW_DIP_x04, Button_Switch_THT:SW_DIP_SPSTx04_Slide_6.7x11.72mm_W7.62mm_P2.54mm_LowProfile, symbol Switch:SW_DIP_x04
- R1, R4, R5, R6, R7: footprint Resistor_THT:R_Axial_DIN0207_L6.3mm_D2.5mm_P7.62mm_Horizontal -> Resistor_SMD:R_1206_3216Metric
- R2, R3: value 330 -> 1k; footprint Resistor_THT:R_Axial_DIN0207_L6.3mm_D2.5mm_P7.62mm_Horizontal -> Resistor_SMD:R_1206_3216Metric
- Y1: value Crystal_GND2 -> 16MHz
- renumbered ESC1 to K0, N1 to K1, N10 to K10, -1 to K11, =1 to K12, BACKSPACE1 to K13, TAB1 to K14, q1 to K15, w1 to K16, e1 to K17, r1 to K18, t1 to K19, N2 to K2, y1 to K20, u1 to K21, i1 to K22, o1 to K23, p1 to K24, [1 to K25, ]1 to K26, \1 to K27, FN1 to K28, a1 to K29, N3 to K3, s1 to K30, d1 to K31, f1 to K32, g1 to K33, h1 to K34, j1 to K35, k1 to K36, l1 to K37, ;1 to K38, '1 to K39, N4 to K4, ENTER1 to K40, SHIFT_LEFT1 to K41, z1 to K42, x1 to K43, c1 to K44, v1 to K45, b1 to K46, n1 to K47, m1 to K48, ,1 to K49, N5 to K5, .1 to K50, /1 to K51, ARROW_UP1 to K52, SHIFT_RIGHT1 to K53, CTRL1 to K54, SUPER1 to K55, ALT_LEFT1 to K56, SPACE1 to K57, ALT_RIGHT1 to K58, ARROW_LEFT1 to K59, N6 to K6, ARROW_DOWN1 to K60, ARROW_RIGHT1 to K61, N7 to K7, N8 to K8, N9 to K9
Connections:
- net labels added: DIP1, DIP2, DIP3, DIP4, LED, RST
- net labels removed: LED_B, LED_G, LED_R
- wire segments 351 -> 376
- no-connect marks 5 -> 3

Commit message: update
Parts:
- added TP1, TP2, TP3: TestPoint_Probe, TestPoint:TestPoint_Pad_D1.0mm, symbol Connector:TestPoint_Probe
Connections:
- wire segments 376 -> 378
Other:
- note added: "6-pin ISP header"
- moved on the sheet: C4
